File: Hardware/tinyPipes v2.6.brd (EAGLE design)
At the start: 59 x 59 mm, 94 parts, among them Q1 CJ2302, Q5 S9013, Q6 S9013, Q7 S9013, U1 TD1410, U2 ICS_V54_SIM900, U3 ATMEGA168, U4 MAX4372, U5 SI4435POWER

Commit message: removed two LEDs and rearranged remaining three for more board space.  Added two more holes for battery leads and a current sense resistor
Parts:
- removed AVRISP: AVR_SPI_PRG_62X3_LOCK, SparkFun:2X3_LOCK
- removed CHARGING, ENABLED: (no value), Discrete:LED-0603
- removed R28, R8: 10k, Discrete:R0603
- added BATTERY+1, BATTERY-1: TINYPIPES_BATTBATT, tinyPipes_v2.5:TINYPIPES_BATT
- added RSENSE1: 0.003, Discrete:R2512
- moved R15 15.2 mm to (6.71, 43.4), turned to 270 degrees
- moved R16 14.3 mm to (5.09, 43.4), turned to 270 degrees
- moved R1 13.9 mm to (3.47, 43.4), turned to 90 degrees
- moved Q6 13.8 mm to (4.19, 36.3), turned to 90 degrees
- moved R13 11.8 mm to (6.79, 36.3), turned to 90 degrees
- moved STATUS 10.9 mm to (6.71, 46.5), turned to 270 degrees
- moved Q5 10.5 mm to (4.19, 39.6), turned to 90 degrees
- moved C8 10.5 mm to (10.2, 37.1)
- moved R21 10.5 mm to (10.2, 38.6)
- moved R3 9.86 mm to (10.2, 35.6), turned to 180 degrees
- moved NETLIGHT 9.60 mm to (5.09, 46.5), turned to 270 degrees
- moved POWER 8.90 mm to (3.47, 46.5), turned to 270 degrees
- moved R14 7.87 mm to (6.80, 39.6), turned to 270 degrees
- moved R20 7.26 mm to (10.2, 40.1)
- moved BATTERY- 3.94 mm to (14.6, 56.4)
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Connections:
- removed net N$10: R8.1, U3.12
- removed net N$14: R28.1, U3.13
- removed net N$18: CHARGING.+, R8.2
- removed net N$24: ENABLED.+, R28.2
- net GND: no longer AVRISP.6, CHARGING.-, ENABLED.-
- net MISO: no longer AVRISP.1
- net MOSI: no longer AVRISP.4
- net RST: no longer AVRISP.5
- net SCK: no longer AVRISP.3
- net VCC: no longer AVRISP.2
Routing:
- net SCK: track 34.2 -> 17.4 mm, vias 0 -> 1
- net N$14: track 15.6 -> 0.00 mm, vias 2 -> 0
- net N$10: track 15.5 -> 0.00 mm, vias 2 -> 0
- net VCC: track 179.2 -> 166.8 mm, vias 11 -> 10
- net MOSI: track 29.5 -> 18.4 mm
- net NETLIGHT: track 79.6 -> 68.7 mm
- net RST: track 49.9 -> 39.9 mm, vias 1 -> 2
- net N$8: track 15.6 -> 5.72 mm
- net STATUS: track 64.8 -> 57.1 mm
- net N$3: track 16.2 -> 8.49 mm
- net MISO: track 28.4 -> 21.2 mm
- net N$24: track 4.65 -> 0.00 mm
- net N$18: track 4.57 -> 0.00 mm
- net N$6: track 3.10 -> 5.52 mm
- net N$5: track 3.10 -> 4.70 mm
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