File: Hardware/tinyPipes v2.6.sch (EAGLE design)
At the start: 94 parts, among them Q1 CJ2302, Q5 S9013, Q6 S9013, Q7 S9013, U1 TD1410, U2 ICS_V54_SIM900, U3 ATMEGA168, U4 MAX4372, U5 SI4435POWER

Commit message: removed two LEDs and rearranged remaining three for more board space.  Added two more holes for battery leads and a current sense resistor
Parts:
- removed AVRISP: AVR_SPI_PRG_62X3_LOCK, SparkFun:AVR_SPI_PRG_62X3_LOCK
- removed CHARGING, ENABLED: (no value), Discrete:LED'0603'
- removed R28, R8: 10k, Discrete:R-0603
- added BATTERY+1, BATTERY-1: TINYPIPES_BATTBATT, tinyPipes_v2.5:TINYPIPES_BATTBATT
- added RSENSE1: 0.003, Discrete:R-2512
Connections:
- removed net N$10: R8.1, U3.PB0(ICP)
- removed net N$14: R28.1, U3.PB1(OC1A)
- removed net N$18: CHARGING.+, R8.2
- removed net N$24: ENABLED.+, R28.2
- net GND: no longer AVRISP.6, CHARGING.-, ENABLED.-
- net MISO: no longer AVRISP.1
- net MOSI: no longer AVRISP.4
- net RST: no longer AVRISP.5
- net SCK: no longer AVRISP.3
- net VCC: no longer AVRISP.2
Changed lines of the file:
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@@
 <?xml version="1.0" encoding="utf-8"?>
 <!DOCTYPE eagle SYSTEM "eagle.dtd">
-<eagle version="6.4">
+<eagle version="6.5.0">
 <drawing>
 <settings>
@@
 <setting verticaltext="up"/>
 </settings>
-<grid distance="50" unitdist="mil" unit="mil" style="lines" multiple="1" display="yes" altdistance="25" altunitdist="mil" altunit="mil"/>
+<grid distance="0.1" unitdist="inch" unit="inch" style="lines" multiple="1" display="no" altdistance="0.01" altunitdist="inch" altunit="inch"/>
 <layers>
 <layer number="1" name="Top" color="4" fill="1" visible="no" active="no"/>
@@
 <part name="ANT1" library="Connector" deviceset="ANTENNA-U-FL" device=""/>
 <part name="U3" library="SparkFun" deviceset="ATMEGA168" device=""/>
-<part name="AVRISP" library="SparkFun" deviceset="AVR_SPI_PRG_6" device="2X3_LOCK"/>
 <part name="P+1" library="supply1" deviceset="VCC" device=""/>
 <part name="P+2" library="supply1" deviceset="VCC" device=""/>
@@
 <part name="PANEL-" library="tinyPipes_v2.5" deviceset="TINYPIPES_BATT" device="PANEL" value="TINYPIPES_BATTPANEL"/>
 <part name="U5" library="tinyPipes" deviceset="SI4435" device="POWER" value="SI4435POWER"/>
-<part name="R8" library="Discrete" deviceset="R*" device="-0603" value="10k"/>
-<part name="R28" library="Discrete" deviceset="R*" device="-0603" value="10k"/>
 <part name="D2" library="diode" deviceset="DIODE-" device="SMB" value="SS54"/>
 <part name="VDD1" library="supply1" deviceset="VDD" device=""/>
@@
 <part name="U$9" library="Power or GND " deviceset="GND_POWER" device=""/>
 <part name="U$11" library="Power or GND " deviceset="GND_POWER" device=""/>
-<part name="U$13" library="Power or GND " deviceset="GND_POWER" device=""/>
 <part name="U$14" library="Power or GND " deviceset="GND_POWER" device=""/>
 <part name="C6" library="Discrete" deviceset="C*" device="-0603" value="100nF"/>
@@
 <part name="U$24" library="Power or GND " deviceset="GND_POWER" device=""/>
 <part name="POWER" library="Discrete" deviceset="LED*" device="'0603'"/>
-<part name="ENABLED" library="Discrete" deviceset="LED*" device="'0603'"/>
-<part name="CHARGING" library="Discrete" deviceset="LED*" device="'0603'"/>
 <part name="STATUS" library="Discrete" deviceset="LED*" device="'0603'"/>
 <part name="NETLIGHT" library="Discrete" deviceset="LED*" device="'0603'"/>
@@
 <part name="F1" library="template" deviceset="FUSE" device="'16R700'"/>
 <part name="X1" library="Discrete" deviceset="CRYSTAL*" device="'5032'"/>
+<part name="BATTERY+1" library="tinyPipes_v2.5" deviceset="TINYPIPES_BATT" device="BATT"/>
+<part name="BATTERY-1" library="tinyPipes_v2.5" deviceset="TINYPIPES_BATT" device="BATT"/>
+<part name="RSENSE1" library="Discrete" deviceset="R*" device="-2512" value="0.003"/>
 </parts>
 <sheets>
@@
 <instance part="U$25" gate="G$1" x="276.86" y="67.31" rot="R270"/>
 <instance part="U3" gate="G$1" x="397.51" y="58.42"/>
-<instance part="AVRISP" gate="G$1" x="491.49" y="66.04"/>
 <instance part="P+1" gate="VCC" x="509.27" y="71.12"/>
 <instance part="P+2" gate="VCC" x="374.65" y="81.28"/>
@@
 <instance part="P+7" gate="VCC" x="434.34" y="146.05"/>
 <instance part="FRAME2" gate="G$1" x="262.89" y="0"/>
-<instance part="R8" gate="R" x="433.07" y="38.1" smashed="yes">
-<attribute name="NAME" x="429.26" y="39.5986" size="1.778" layer="95"/>
-<attribute name="VALUE" x="434.34" y="39.878" size="1.778" layer="96"/>
-</instance>
-<instance part="R28" gate="R" x="433.07" y="35.56" smashed="yes">
-<attribute name="NAME" x="436.88" y="35.56" size="1.778" layer="95"/>
-<attribute name="VALUE" x="443.23" y="35.56" size="1.778" layer="96"/>
-</instance>
 <instance part="P+8" gate="VCC" x="356.87" y="73.66"/>
 <instance part="R1" gate="R" x="341.63" y="50.8"/>
@@
 <instance part="U$9" gate="G$1" x="360.68" y="49.53"/>
 <instance part="U$11" gate="G$1" x="373.38" y="25.4"/>
-<instance part="U$13" gate="G$1" x="452.12" y="30.48"/>
 <instance part="U$14" gate="G$1" x="509.27" y="63.5" rot="R90"/>
 <instance part="C6" gate="C" x="34.29" y="-91.44" rot="R90"/>
@@
 <instance part="U$24" gate="G$1" x="448.31" y="135.89"/>
 <instance part="POWER" gate="LED" x="346.71" y="57.15" rot="R270"/>
-<instance part="ENABLED" gate="LED" x="445.77" y="31.75"/>
-<instance part="CHARGING" gate="LED" x="445.77" y="40.64"/>
 <instance part="STATUS" gate="LED" x="200.66" y="134.62" rot="R180"/>
 <instance part="NETLIGHT" gate="LED" x="199.39" y="114.3" rot="R180"/>
@@
 <instance part="F1" gate="F" x="149.86" y="-123.19"/>
 <instance part="X1" gate="X" x="372.11" y="54.61" rot="R90"/>
+<instance part="BATTERY+1" gate="G$1" x="140.97" y="-110.49" rot="R180"/>
+<instance part="BATTERY-1" gate="G$1" x="140.97" y="-115.57" rot="R180"/>
+<instance part="RSENSE1" gate="R" x="151.13" y="-111.76" smashed="yes" rot="R90">
+<attribute name="NAME" x="147.0914" y="-115.57" size="1.778" layer="95" rot="R90"/>
+<attribute name="VALUE" x="149.352" y="-114.3" size="1.778" layer="96" rot="R90"/>
+</instance>
 </instances>
 <busses>
@@
 </segment>
 <segment>
-<pinref part="AVRISP" gate="G$1" pin="6"/>
 <wire x1="501.65" y1="63.5" x2="509.27" y2="63.5" width="0.1524" layer="91"/>
 <pinref part="U$14" gate="G$1" pin="GND"/>
@@
 <wire x1="360.68" y1="49.53" x2="360.68" y2="53.34" width="0.1524" layer="91"/>
 <junction x="360.68" y="53.34"/>
-</segment>
-<segment>
-<wire x1="449.58" y1="40.64" x2="452.12" y2="40.64" width="0.1524" layer="91"/>
-<wire x1="452.12" y1="40.64" x2="452.12" y2="31.75" width="0.1524" layer="91"/>
-<wire x1="452.12" y1="31.75" x2="452.12" y2="30.48" width="0.1524" layer="91"/>
-<wire x1="449.58" y1="31.75" x2="452.12" y2="31.75" width="0.1524" layer="91"/>
-<junction x="452.12" y="31.75"/>
-<pinref part="U$13" gate="G$1" pin="GND"/>
-<pinref part="ENABLED" gate="LED" pin="-"/>
-<pinref part="CHARGING" gate="LED" pin="-"/>
 </segment>
 <segment>
@@
 </segment>
 <segment>
-<pinref part="AVRISP" gate="G$1" pin="2"/>
 <pinref part="P+1" gate="VCC" pin="VCC"/>
 <wire x1="509.27" y1="68.58" x2="501.65" y2="68.58" width="0.1524" layer="91"/>
@@
 <net name="MOSI" class="0">
 <segment>
-<pinref part="AVRISP" gate="G$1" pin="4"/>
 <wire x1="501.65" y1="66.04" x2="509.27" y2="66.04" width="0.1524" layer="91"/>
 <label x="511.81" y="66.04" size="1.778" layer="95"/>
@@
 <net name="MISO" class="0">
 <segment>
-<pinref part="AVRISP" gate="G$1" pin="1"/>
 <wire x1="483.87" y1="68.58" x2="476.25" y2="68.58" width="0.1524" layer="91"/>
 <label x="468.63" y="68.58" size="1.778" layer="95"/>
@@
 <net name="SCK" class="0">
 <segment>
-<pinref part="AVRISP" gate="G$1" pin="3"/>
 <wire x1="483.87" y1="66.04" x2="476.25" y2="66.04" width="0.1524" layer="91"/>
 <label x="468.63" y="66.04" size="1.778" layer="95"/>
@@
 <net name="RST" class="0">
 <segment>
-<pinref part="AVRISP" gate="G$1" pin="5"/>
 <wire x1="483.87" y1="63.5" x2="476.25" y2="63.5" width="0.1524" layer="91"/>
 <label x="468.63" y="63.5" size="1.778" layer="95"/>
@@
 <wire x1="76.2" y1="-125.73" x2="81.28" y2="-125.73" width="0.1524" layer="91"/>
 <junction x="76.2" y="-125.73"/>
-</segment>
-</net>
-<net name="N$10" class="1">
-<segment>
-<pinref part="U3" gate="G$1" pin="PB0(ICP)"/>
-<pinref part="R8" gate="R" pin="1"/>
-<wire x1="429.26" y1="38.1" x2="422.91" y2="38.1" width="0.1524" layer="91"/>
-</segment>
-</net>
-<net name="N$14" class="1">
-<segment>
-<pinref part="U3" gate="G$1" pin="PB1(OC1A)"/>
-<pinref part="R28" gate="R" pin="1"/>
-<wire x1="429.26" y1="35.56" x2="422.91" y2="35.56" width="0.1524" layer="91"/>
 </segment>
 </net>
@@
 </segment>
 </net>
-<net name="N$18" class="0">
-<segment>
-<pinref part="R8" gate="R" pin="2"/>
-<wire x1="441.96" y1="40.64" x2="436.88" y2="38.1" width="0.1524" layer="91"/>
-<pinref part="CHARGING" gate="LED" pin="+"/>
-</segment>
-</net>
-<net name="N$24" class="0">
-<segment>
-<pinref part="R28" gate="R" pin="2"/>
-<wire x1="441.96" y1="31.75" x2="436.88" y2="35.56" width="0.1524" layer="91"/>
-<pinref part="ENABLED" gate="LED" pin="+"/>
-</segment>
-</net>
