File: Hardware/tinyPipes.sch (EAGLE design)
At the start: 107 parts, among them Q1 CJ2302, Q2 CJ2302, Q3 CJ2302, Q4 BSS84, Q5 S9013, Q6 S9013, Q7 S9013, U1 TD1410, U2 ICS_V54_SIM900, U3 ATMEGA168MLF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

Commit message: stashing latest changes -- still a work in progress
Parts:
- removed Q3: CJ2302, Discrete:MOSFET-N'SOT23'
- removed R23, R8: 10k, rcl:R-US_R0201
- added R29: 10k, rcl:R-US_R0201
Connections:
- net LOW_SIDE renamed PILLOWTALK_LOW_SIDE
- removed net HIGH_SIDE: Q3.G, R8.2, U3.PB0(ICP)
- removed net PFET_GATE: Q3.D, Q4.G, R23.1
- new net PILLOWTALK_HIGH_SIDE: Q4.G, R29.1, U3.PB0(ICP)
- net BATTERY: no longer R23.2
- net GND: no longer Q3.S, R8.1
- net VCC: now also R29.2
Changed lines of the file:
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@@
 <setting verticaltext="up"/>
 </settings>
-<grid distance="0.1" unitdist="inch" unit="inch" style="lines" multiple="1" display="no" altdistance="0.01" altunitdist="inch" altunit="inch"/>
+<grid distance="0.05" unitdist="inch" unit="inch" style="lines" multiple="1" display="no" altdistance="0.01" altunitdist="inch" altunit="inch"/>
 <layers>
 <layer number="1" name="Top" color="4" fill="1" visible="no" active="no"/>
@@
 <part name="U$5" library="Power or GND " deviceset="GND_POWER" device=""/>
 <part name="C23" library="Discrete" deviceset="CAP*" device="-AVX-D" value="470uF 6.3V"/>
-<part name="R23" library="rcl" deviceset="R-US_" device="R0201" value="10k"/>
-<part name="GND6" library="supply1" deviceset="GND" device=""/>
 <part name="FRAME4" library="frames" deviceset="A4L-LOC" device=""/>
 <part name="Q2" library="Discrete" deviceset="MOSFET-N" device="'SOT23'" value="CJ2302"/>
-<part name="Q3" library="Discrete" deviceset="MOSFET-N" device="'SOT23'" value="CJ2302"/>
 <part name="U$1" library="tinyPipes" deviceset="5A-10UH-INDUCTOR" device=""/>
-<part name="R8" library="rcl" deviceset="R-US_" device="R0201" value="10k"/>
 <part name="R28" library="rcl" deviceset="R-US_" device="R0201" value="10k"/>
 <part name="U3" library="tinyPipes" deviceset="ATMEGA168" device="MLF" value="ATMEGA168MLF"/>
@@
 <part name="C5" library="rcl" deviceset="C-US" device="C0402" value="100nF"/>
 <part name="C9" library="rcl" deviceset="C-US" device="C0402" value="100nF"/>
+<part name="R29" library="rcl" deviceset="R-US_" device="R0201" value="10k"/>
 </parts>
 <sheets>
@@
 <wire x1="241.3" y1="-151.13" x2="119.38" y2="-151.13" width="0.1524" layer="94"/>
 <wire x1="119.38" y1="-151.13" x2="119.38" y2="-62.23" width="0.1524" layer="94"/>
-<text x="367.03" y="-75.946" size="1.27" layer="91">5A, 10uH choke</text>
+<text x="368.3" y="-77.216" size="1.27" layer="91">5A, 10uH choke</text>
 </plain>
 <instances>
@@
 <instance part="U$5" gate="G$1" x="360.68" y="-113.03"/>
 <instance part="C23" gate="C" x="387.35" y="-86.36"/>
-<instance part="R23" gate="G$1" x="431.8" y="-77.47" rot="R90"/>
-<instance part="GND6" gate="1" x="431.8" y="-102.87"/>
 <instance part="FRAME4" gate="G$1" x="261.62" y="-180.34"/>
 <instance part="Q2" gate="MOS" x="360.68" y="-99.06"/>
-<instance part="Q3" gate="MOS" x="431.8" y="-87.63"/>
-<instance part="U$1" gate="G$1" x="375.92" y="-80.01" rot="R90"/>
-<instance part="R8" gate="G$1" x="426.72" y="-95.25" rot="R90"/>
+<instance part="U$1" gate="G$1" x="375.92" y="-80.01" smashed="yes" rot="R90">
+<attribute name="NAME" x="381" y="-81.28" size="1.778" layer="95" rot="R180"/>
+</instance>
 <instance part="R28" gate="G$1" x="354.33" y="-106.68" rot="R90"/>
 <instance part="U3" gate="G$1" x="397.51" y="58.42"/>
 <instance part="Q4" gate="G$1" x="360.68" y="-87.63"/>
-<instance part="P+12" gate="VCC" x="360.68" y="-77.47"/>
+<instance part="P+12" gate="VCC" x="360.68" y="-72.39"/>
 <instance part="B+" gate="G$1" x="154.94" y="-114.3" rot="R180"/>
 <instance part="C4" gate="G$1" x="407.67" y="127" smashed="yes">
@@
 <attribute name="VALUE" x="421.386" y="131.699" size="1.778" layer="96"/>
 </instance>
+<instance part="R29" gate="G$1" x="351.79" y="-80.01" rot="R90"/>
 </instances>
 <busses>
@@
 <pinref part="R28" gate="G$1" pin="1"/>
 </segment>
-<segment>
-<pinref part="GND6" gate="1" pin="GND"/>
-<wire x1="431.8" y1="-100.33" x2="431.8" y2="-92.71" width="0.1524" layer="91"/>
-<wire x1="426.72" y1="-100.33" x2="431.8" y2="-100.33" width="0.1524" layer="91"/>
-<junction x="431.8" y="-100.33"/>
-<pinref part="Q3" gate="MOS" pin="S"/>
-<pinref part="R8" gate="G$1" pin="1"/>
-</segment>
 </net>
 <net name="SIM_DATA" class="0">
@@
 </segment>
 <segment>
-<pinref part="R23" gate="G$1" pin="2"/>
-<wire x1="431.8" y1="-72.39" x2="434.34" y2="-72.39" width="0.1524" layer="91"/>
-<label x="434.34" y="-72.39" size="1.27" layer="95" xref="yes"/>
-</segment>
-<segment>
 <wire x1="383.54" y1="-80.01" x2="392.43" y2="-80.01" width="0.1524" layer="91"/>
 <wire x1="392.43" y1="-80.01" x2="392.43" y2="-86.36" width="0.1524" layer="91"/>
@@
 </segment>
 </net>
-<net name="LOW_SIDE" class="0">
-<segment>
-<wire x1="422.91" y1="76.2" x2="427.99" y2="76.2" width="0.1524" layer="91"/>
-<label x="427.99" y="76.2" size="1.27" layer="95" xref="yes"/>
-<pinref part="U3" gate="G$1" pin="PC3(ADC3)"/>
-</segment>
-<segment>
-<pinref part="Q2" gate="MOS" pin="G"/>
-<pinref part="R28" gate="G$1" pin="2"/>
-<wire x1="355.6" y1="-99.06" x2="354.33" y2="-99.06" width="0.1524" layer="91"/>
-<wire x1="354.33" y1="-99.06" x2="354.33" y2="-101.6" width="0.1524" layer="91"/>
-<wire x1="354.33" y1="-99.06" x2="346.71" y2="-99.06" width="0.1524" layer="91"/>
-<junction x="354.33" y="-99.06"/>
-<label x="347.98" y="-99.06" size="1.27" layer="95" rot="R180" xref="yes"/>
-</segment>
-</net>
-<net name="PFET_GATE" class="0">
-<segment>
-<pinref part="R23" gate="G$1" pin="1"/>
-<wire x1="431.8" y1="-82.55" x2="427.99" y2="-82.55" width="0.1524" layer="91"/>
-<label x="427.99" y="-82.55" size="1.27" layer="95" rot="R180" xref="yes"/>
-<pinref part="Q3" gate="MOS" pin="D"/>
-<junction x="431.8" y="-82.55"/>
-</segment>
-<segment>
-<pinref part="Q4" gate="G$1" pin="G"/>
-<wire x1="355.6" y1="-85.09" x2="351.79" y2="-85.09" width="0.1524" layer="91"/>
-<label x="350.52" y="-85.09" size="1.27" layer="95" rot="R180" xref="yes"/>
-</segment>
-</net>
-<net name="HIGH_SIDE" class="0">
-<segment>
-<wire x1="422.91" y1="38.1" x2="425.45" y2="38.1" width="0.1524" layer="91"/>
-<label x="425.45" y="38.1" size="1.27" layer="95" xref="yes"/>
-<pinref part="U3" gate="G$1" pin="PB0(ICP)"/>
-</segment>
-<segment>
-<pinref part="Q3" gate="MOS" pin="G"/>
-<pinref part="R8" gate="G$1" pin="2"/>
-<wire x1="426.72" y1="-87.63" x2="426.72" y2="-90.17" width="0.1524" layer="91"/>
-<wire x1="426.72" y1="-87.63" x2="420.37" y2="-87.63" width="0.1524" layer="91"/>
-<junction x="426.72" y="-87.63"/>
-<label x="420.37" y="-87.63" size="1.27" layer="95" rot="R180" xref="yes"/>
-</segment>
-</net>
 <net name="VCC" class="0">
 <segment>
 <pinref part="Q4" gate="G$1" pin="S"/>
-<wire x1="360.68" y1="-80.01" x2="360.68" y2="-82.55" width="0.1524" layer="91"/>
+<wire x1="360.68" y1="-74.93" x2="360.68" y2="-82.55" width="0.1524" layer="91"/>
 <pinref part="P+12" gate="VCC" pin="VCC"/>
+<pinref part="R29" gate="G$1" pin="2"/>
+<wire x1="360.68" y1="-74.93" x2="351.79" y2="-74.93" width="0.1524" layer="91"/>
+<junction x="360.68" y="-74.93"/>
 </segment>
 </net>
@@
 </segment>
 </net>
+<net name="PILLOWTALK_HIGH_SIDE" class="0">
+<segment>
+<pinref part="Q4" gate="G$1" pin="G"/>
+<wire x1="355.6" y1="-85.09" x2="351.79" y2="-85.09" width="0.1524" layer="91"/>
+<label x="342.9" y="-85.09" size="1.27" layer="95" rot="R180" xref="yes"/>
+<pinref part="R29" gate="G$1" pin="1"/>
+<wire x1="351.79" y1="-85.09" x2="344.17" y2="-85.09" width="0.1524" layer="91"/>
+<junction x="351.79" y="-85.09"/>
+</segment>
+<segment>
+<wire x1="422.91" y1="38.1" x2="425.45" y2="38.1" width="0.1524" layer="91"/>
+<label x="425.45" y="38.1" size="1.27" layer="95" xref="yes"/>
+<pinref part="U3" gate="G$1" pin="PB0(ICP)"/>
+</segment>
+</net>
+<net name="PILLOWTALK_LOW_SIDE" class="0">
+<segment>
+<pinref part="Q2" gate="MOS" pin="G"/>
+<pinref part="R28" gate="G$1" pin="2"/>
+<wire x1="355.6" y1="-99.06" x2="354.33" y2="-99.06" width="0.1524" layer="91"/>
+<wire x1="354.33" y1="-99.06" x2="354.33" y2="-101.6" width="0.1524" layer="91"/>
+<wire x1="354.33" y1="-99.06" x2="344.17" y2="-99.06" width="0.1524" layer="91"/>
+<junction x="354.33" y="-99.06"/>
+<label x="342.9" y="-99.06" size="1.27" layer="95" rot="R180" xref="yes"/>
+</segment>
+<segment>
+<wire x1="422.91" y1="76.2" x2="427.99" y2="76.2" width="0.1524" layer="91"/>
+<label x="427.99" y="76.2" size="1.27" layer="95" xref="yes"/>
+<pinref part="U3" gate="G$1" pin="PC3(ADC3)"/>
+</segment>
+</net>
