File: Hardware/tinyPipes.sch (EAGLE design)
At the start: 109 parts, among them J1 Micro-USB connector, Q1 CJ2302, Q2 BSS84, Q5 S9013, Q6 S9013, Q7 S9013, Q8 BSS123, Q9 BSS123, U1 TD1410, U2 ICS_V54_SIM900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

Commit message: tinyPipes v3.1
Parts:
- R11: value (none) -> 10k
Changed lines of the file:
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@@
 <setting verticaltext="up"/>
 </settings>
-<grid distance="0.05" unitdist="inch" unit="inch" style="lines" multiple="1" display="no" altdistance="0.01" altunitdist="inch" altunit="inch"/>
+<grid distance="0.1" unitdist="inch" unit="inch" style="lines" multiple="1" display="no" altdistance="0.01" altunitdist="inch" altunit="inch"/>
 <layers>
 <layer number="1" name="Top" color="4" fill="1" visible="no" active="no"/>
@@
 <part name="D1" library="diode" deviceset="ZENER-DIODE" device="SOT23" value="5v"/>
 <part name="Q9" library="transistor-small-signal" deviceset="BSS123" device=""/>
-<part name="R11" library="rcl" deviceset="R-US_" device="R0402"/>
+<part name="R11" library="rcl" deviceset="R-US_" device="R0402" value="10k"/>
 <part name="GND5" library="supply1" deviceset="GND" device=""/>
 <part name="J1" library="OPL Eagle Library" deviceset="MICRO-USB-5P" device="-340015001" value="Micro-USB connector"/>
