File: Hardware/proto/tinyPipes v2.6.brd (EAGLE design)
At the start: 59 x 59 mm, 98 parts, among them Q1 CJ2302, Q5 S9013, Q6 S9013, Q7 S9013, U1 TD1410, U2 ICS_V54_SIM900, U3 ATMEGA168, U4 MAX4372, U5 SI4435POWER, U6 MAX4372

Commit message: finished routing proto board
Parts:
- added BM, BP: TINYPIPES_BATTSBATT, tinyPipes v2.6:TINYPIPES_SBATT
- added Q2: IRFR5305, transistor-power:D-PAK_TO252AA
- added Q3: CJ2302, Discrete:SOT23
- added R28: 10k, Discrete:R0603
- added R29: 100k, Discrete:R0603
- added R30: 1k, Discrete:R0603
- F1, F2: device template:0210 -> tinyPipes v2.6:0210
- moved F2 40.5 mm to (6.73, 53.2), turned to 90 degrees
- moved OUT+ 23.3 mm to (3.68, 50.8)
- moved B+ 18.0 mm to (30.7, 56.4)
- moved RSENSE1 1.91 mm to (24.6, 56.4), turned to 180 degrees
- moved C13 1.14 mm to (26.5, 40.5)
- moved C14 1.14 mm to (26.5, 37.5)
- moved R24 1.14 mm to (26.6, 39.0)
- moved R25 1.14 mm to (26.5, 42.0)
- moved R26 1.14 mm to (26.6, 34.4)
- moved R27 1.14 mm to (26.6, 35.9)
- moved RSENSE 0.92 mm to (34.6, 43.4)
- moved F1 0.76 mm to (31.4, 52.1)
Connections:
- new net BATT_EN: R30.2, U3.28
- new net BV+: BP.P$1, R24.2
- new net BV-: BM.P$1, U3.27
- new net N$18: F2.2, Q2.4
- new net N$19: F2.1, OUT+.1
- new net N$20: Q2.1, Q3.3, R28.1
- new net N$21: Q3.1, R29.2, R30.1
- net BATT: now also B+.1, R23.1; no longer R8.1
- net BATTERY: no longer R24.2
- net GND: now also Q3.2, R29.1
- net N$10: now also Q2.3, R28.2, R8.1; no longer OUT+.1, R23.1
Routing:
- net BATT_EN: track 0.00 -> 26.1 mm, vias 0 -> 2
- net BV-: track 0.00 -> 7.94 mm
- net N$20: track 0.00 -> 7.21 mm
- net BATTERY: track 55.4 -> 50.3 mm, vias 1 -> 3
- net N$21: track 0.00 -> 3.05 mm
- net BV+: track 0.00 -> 2.65 mm
- net N$10: track 3.68 -> 5.33 mm
- net BATTERY_VOLTAGE: track 8.80 -> 10.3 mm
- net RSENSE-: track 14.7 -> 15.9 mm
- net RSENSE+: track 17.8 -> 19.1 mm
- net PANEL_VOLTAGE: track 7.56 -> 8.70 mm
- net VCC: track 165.1 -> 164.3 mm
- net BATTERY_CURRENT: track 15.6 -> 15.7 mm, vias 2 -> 0
- net GND: vias 163 -> 167
- added copper zone on layer 1, net BATT
- added copper zone on layer 1, net N$18
- added copper zone on layer 16, net N$18
- added copper zone on layer 1, net N$19
- added copper zone on layer 16, net N$19
