File: Hardware/proto/tinyPipes v2.6.sch (EAGLE design)
At the start: 98 parts, among them Q1 CJ2302, Q5 S9013, Q6 S9013, Q7 S9013, U1 TD1410, U2 ICS_V54_SIM900, U3 ATMEGA168, U4 MAX4372, U5 SI4435POWER, U6 MAX4372

Commit message: finished routing proto board
Parts:
- added BM, BP: TINYPIPES_BATTSBATT, tinyPipes v2.6:TINYPIPES_BATTSBATT
- added Q2: IRFR5305, transistor-power:IRFR5305
- added Q3: CJ2302, Discrete:MOSFET-N'SOT23'
- added R28: 10k, Discrete:R-0603
- added R29: 100k, Discrete:R-0603
- added R30: 1k, Discrete:R-0603
- F1, F2: device template:FUSE'16R700' -> tinyPipes v2.6:FUSE16R700
Connections:
- new net BATT_EN: R30.2, U3.PC5(ADC5/SCL)
- new net BV+: BP.P$1, R24.2
- new net BV-: BM.P$1, U3.PC4(ADC4/SDA)
- new net N$18: F2.2, Q2.D
- new net N$19: F2.1, OUT+.P$1
- new net N$20: Q2.G, Q3.D, R28.1
- new net N$21: Q3.G, R29.2, R30.1
- net BATT: now also B+.P$1, R23.1; no longer R8.1
- net BATTERY: no longer R24.2
- net GND: now also Q3.S, R29.1
- net N$10: now also Q2.S, R28.2, R8.1; no longer OUT+.P$1, R23.1
Other:
- moved on the sheet: B+, B-, D4, F2, OUT+, OUT-
