File: Hardware/demo/demo.brd (EAGLE design)
At the start: 59 x 59 mm, 69 parts, among them Q1 CJ2302, Q2 CJ2302, Q3 CJ2302, Q4 CJ2302, Q5 CJ2302, Q6 CJ2302, Q7 BSS84, Q8 BSS123, Q9 BSS123, U1 TD1410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

Commit message: netRequest is working really well -- I have the time between requests down to about 5 seconds
Parts:
- D1: value (none) -> 5v
Changed lines of the file:
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@@
 <element name="L1-" library="tinyPipes_v2.5" package="TINYPIPES_BATT" value="TINYPIPES_BATTBATT" x="24.13" y="32.004"/>
 <element name="R2" library="Discrete" package="R0603" value="10k" x="13.208" y="37.592" rot="R90"/>
-<element name="D1" library="diode" package="SOD80C" value="" x="15.24" y="36.83" rot="R270"/>
+<element name="D1" library="diode" package="SOD80C" value="5v" x="15.24" y="36.83" rot="R270"/>
 <element name="L2+" library="tinyPipes_v2.5" package="TINYPIPES_BATT" value="TINYPIPES_BATTBATT" x="5.842" y="45.72"/>
 <element name="L2-" library="tinyPipes_v2.5" package="TINYPIPES_BATT" value="TINYPIPES_BATTBATT" x="5.588" y="53.594"/>
