File: Hardware/demo/demo.sch (EAGLE design)
At the start: 69 parts, among them Q1 CJ2302, Q2 CJ2302, Q3 CJ2302, Q4 CJ2302, Q5 CJ2302, Q6 CJ2302, Q7 BSS84, Q8 BSS123, Q9 BSS123, U1 TD1410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

Commit message: netRequest is working really well -- I have the time between requests down to about 5 seconds
Parts:
- D1: value (none) -> 5v
Changed lines of the file:
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@@
 <setting verticaltext="up"/>
 </settings>
-<grid distance="0.05" unitdist="inch" unit="inch" style="lines" multiple="1" display="no" altdistance="0.01" altunitdist="inch" altunit="inch"/>
+<grid distance="0.1" unitdist="inch" unit="inch" style="lines" multiple="1" display="no" altdistance="0.01" altunitdist="inch" altunit="inch"/>
 <layers>
 <layer number="1" name="Top" color="4" fill="1" visible="no" active="no"/>
@@
 <part name="R2" library="Discrete" deviceset="R*" device="-0603" value="10k"/>
 <part name="U$8" library="Power or GND " deviceset="GND_POWER" device=""/>
-<part name="D1" library="diode" deviceset="ZENER-DIODE" device="SOD80C"/>
+<part name="D1" library="diode" deviceset="ZENER-DIODE" device="SOD80C" value="5v"/>
 <part name="L2+" library="tinyPipes_v2.5" deviceset="TINYPIPES_BATT" device="BATT"/>
 <part name="L2-" library="tinyPipes_v2.5" deviceset="TINYPIPES_BATT" device="BATT"/>
