File: Hardware/tinyTinyPipes/tinyPipes-tinyComponents.sch (EAGLE design)
At the start: 108 parts, among them Q1 CJ2302, Q2 IRFR5305, Q3 CJ2302, Q5 S9013, Q6 S9013, Q7 S9013, U1 TD1410, U2 ICS_V54_SIM900, U3 ATMEGA168, U4 MAX4372, U5 SI4435POWER, U6 MAX4372

Commit message: netRequest is working really well -- I have the time between requests down to about 5 seconds
Parts:
- added C26: 0.1uF, rcl:C-USC0402
- added R31, R32: 4.7k, rcl:R-US_R0201
- added U7: EEPROM-I2CSMD, SparkFun-DigitalIC:EEPROM-I2CSMD
- C1, C16: device rcl:C-USC0402 -> rcl:C-USC0201
- R1: device Discrete:R-0603 -> rcl:R-US_R0201
Connections:
- removed net BATT: B+.P$1, R23.1, RSENSE1.1
- removed net N$10: F1.1, Q2.S, R28.2, R8.1, RSENSE1.2
- new net DEK: Q2.S, R28.2, R8.1, RSENSE1.1
- new net N$23: B+.P$1, F1.1, R23.1, RSENSE1.2
- new net SCL: R31.1, U3.PC5(ADC5/SCL), U7.SCL
- new net SDA: R32.1, U3.PC4(ADC4/SDA), U7.SDA
- new net WP: U3.PB1(OC1A), U7.WP
- net BATTERY_VOLTAGE: now also C13.1; no longer C13.2
- net BATT_EN: now also U3.ADC7; no longer U3.PC5(ADC5/SCL)
- net BV-: now also U3.ADC6; no longer U3.PC4(ADC4/SDA)
- net GND: now also C13.2, C14.2, C26.2, U7.A0, U7.A1, U7.A2, U7.VSS; no longer C13.1, C14.1
- net PANEL_VOLTAGE: now also C14.1; no longer C14.2
- net VCC: now also C26.1, R31.2, R32.2, U7.VCC
Other:
- moved on the sheet: B+, BATTERY, C1, C11, C13, C14, C17, C18, C23, C24, C25, C3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

Commit message: pushing up tinyComponents PCB and various firmware changes
Parts:
- removed C25: 100nF, rcl:C-USC0402
- removed F2: (no value), tinyPipes v2.6:FUSE16R700
- removed OUT+, OUT-: TINYPIPES_BATTBATT, tinyPipes v2.6:TINYPIPES_BATTBATT
- removed R29: 100k, rcl:R-US_R0201
- removed R30: 1k, rcl:R-US_R0201
- removed RSENSE1: 0.003, 1%, Discrete:R-2512
- removed U6: MAX4372, tinyPipes:MAX4372
- added D1: SS54, diode:DIODE-SMB
- added Q4: BSS84, transistor-small-signal:BSS84
- added U$1: INDUCTOR, tinyPipes:INDUCTOR
- C23: value 100nF -> 470uF 6.3V; device rcl:C-USC0402 -> Discrete:CAP-AVX-D
- C4: value 10uF -> 10uF; device rcl:C-USC0402 -> rcl:C-USC0805
- Q2: value IRFR5305 -> CJ2302; device transistor-power:IRFR5305 -> Discrete:MOSFET-N'SOT23'
- U3: value ATMEGA168 -> ATMEGA168MLF; device SparkFun:ATMEGA168 -> tinyPipes:ATMEGA168MLF
- X1: value (none) -> 16mhz; device Discrete:CRYSTAL'5032' -> tinyPipes:CRYSTAL
Connections:
- removed net BATTERY_CURRENT: U3.PC3(ADC3), U6.OUT
- removed net BATT_EN: R30.2, U3.ADC7
- removed net DEK: Q2.S, R28.2, R8.1, RSENSE1.1
- removed net N$14: C25.2, R8.2, U6.RSENSE-
- removed net N$18: F2.2, Q2.D
- removed net N$19: F2.1, OUT+.P$1
- removed net N$20: Q2.G, Q3.D, R28.1
- removed net N$21: Q3.G, R29.2, R30.1
- removed net N$23: B+.P$1, F1.1, R23.1, RSENSE1.2
- new net B+: B+.P$1, F1.1
- new net B-: B-.P$1, D4.A
- new net HIGH_SIDE: Q3.G, R8.2, U3.PB0(ICP)
- new net LOW_SIDE: Q2.G, R28.2, U3.PC3(ADC3)
- new net PFET_GATE: Q3.D, Q4.G, R23.1
- new net VROUTE: C17.2, C18.2, C19.2, C2.+, C21.2, C22.2, C26.1, C3.+, C4.1, C5.1, C7.2, C9.1, L1.2, NETLIGHT.+, POWER.+, R3.2, R31.2, R32.2, R6.2, STATUS.+, TTL.4, U2.VBAT@0, U2.VBAT@1, U2.VBAT@2, U3.AREF, U3.AVCC, U3.VCC@1, U3.VCC@2, U7.VCC, VCC.TP
- net BATTERY: now also C23.-, R23.2, U$1.2
- net BV-: no longer U3.ADC6
- net GND: now also C4.2, C5.2, C9.2, Q2.S, R28.1, R8.1; no longer B-.P$1, C23.2, C25.1, C4.1, C5.1, C9.1, D4.A, OUT-.P$1, R29.1, U6.GND
- net N$17: now also C23.+, Q2.D, Q4.D; no longer C23.1, R23.2, U6.RSENSE+
- net PANEL: now also D1.A; no longer U6.VCC
- net VCC: now also Q4.S, U$1.1; no longer C17.2, C18.2, C19.2, C2.+, C21.2, C22.2, C26.1, C3.+, C4.2, C5.2, C7.2, C9.2, L1.2, NETLIGHT.+, POWER.+, R3.2, R31.2, R32.2, R6.2, STATUS.+, TTL.4, U2.VBAT@0, U2.VBAT@1, U2.VBAT@2, U3.AREF, U3.AVCC, U3.VCC@1, U3.VCC@2, U7.VCC, VCC.TP
- net VDD: now also D1.C
Other:
- note added: "5A, 10uH choke"
- moved on the sheet: B+, C4, C5, C9, Q3, R23, R28, R8
